File: fla-lampi/fla-lampi.kicad_sch (KiCad schematic)
At the start: 6 parts, among them J1 Screw_Terminal_01x03_P3.5mm, M1 Module_XIAO-RP2040_SocketSMD, SW1 BUTTON_B3SN, SW2 BUTTON_B3SN

Commit message: Bretti
Parts:
- removed J1: Screw_Terminal_01x03_P3.5mm, fab:TerminalBlock_OnShore_1x03_P3.50mm_Horizontal, symbol fab:Screw_Terminal_01x03_P3.5mm
- removed M1: Module_XIAO-RP2040_SocketSMD, fab:SeeedStudio_XIAO_SocketSMD, symbol fab:Module_XIAO-RP2040_SocketSMD
- added J2: Conn_PinHeader_1x03_P2.54mm_Horizontal_SMD, fab:PinHeader_1x03_P2.54mm_Horizontal_SMD, symbol fab:Conn_PinHeader_1x03_P2.54mm_Horizontal_SMD
- added M2: Module_XIAO-RP2040, fab:SeeedStudio_XIAO_RP2040, symbol fab:Module_XIAO-RP2040
Connections:
- net A0: now also M2.1 (D0)
- net A1: now also M2.2 (D1)
- net A10: now also M2.11 (D10)
- net A2: now also M2.3 (D2)
- net A3: now also M2.4 (D3)
- net A6: now also J2.1 (Pin_1), M2.7 (D6)
- net A7: now also M2.8 (D7)
- net A8: now also M2.9 (D8)
- net A9: now also M2.10 (D9)
- net GND: now also J2.3 (Pin_3), M2.13 (GND)
- net PWR_3V3: now also M2.12 (3V3)
- net PWR_5V: now also J2.2 (Pin_2), M2.14 (5V)
- net SCL: now also M2.6 (D5)
- net SDA: now also M2.5 (D4)
Changed lines of the file:
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@@
+    (stroke (width 0) (type default))
+  )
+  (wire (pts (xy 105.918 59.944) (xy 96.393 59.944))
     (stroke (width 0) (type default))
   )
@@
     (stroke (width 0) (type default))
   )
-  (wire (pts (xy 96.3676 57.404) (xy 98.044 57.404))
-    (stroke (width 0) (type default))
-  )
   (wire (pts (xy 127.127 62.992) (xy 128.524 62.992))
     (stroke (width 0) (type default))
@@
     (stroke (width 0) (type default))
   )
+  (wire (pts (xy 105.918 59.309) (xy 105.918 59.944))
+    (stroke (width 0) (type default))
+  )
   (wire (pts (xy 141.224 45.339) (xy 141.224 47.752))
     (stroke (width 0) (type default))
@@
     (stroke (width 0) (type default))
   )
-  (wire (pts (xy 98.044 55.753) (xy 98.044 57.404))
-    (stroke (width 0) (type default))
-  )
   (wire (pts (xy 127.127 78.232) (xy 128.524 78.232))
     (stroke (width 0) (type default))
@@
     (stroke (width 0) (type default))
   )
-  (wire (pts (xy 141.224 83.312) (xy 141.224 84.963))
-    (stroke (width 0) (type default))
-  )
-  (wire (pts (xy 104.5464 59.944) (xy 104.5464 61.976))
-    (stroke (width 0) (type default))
-  )
-  (wire (pts (xy 96.3676 59.944) (xy 104.5464 59.944))
-    (stroke (width 0) (type default))
-  )
   (wire (pts (xy 172.212 106.68) (xy 172.212 101.219))
     (stroke (width 0) (type default))
@@
     )
   )
-  (global_label "A8" (shape input) (at 96.3676 62.484 0) (fields_autoplaced)
+  (global_label "A6" (shape input) (at 96.393 57.404 0) (fields_autoplaced)
     (effects (font (size 1.27 1.27)) (justify left))
-    (property "Intersheetrefs" "${INTERSHEET_REFS}" (at 101.6509 62.484 0)
+    (property "Intersheetrefs" "${INTERSHEET_REFS}" (at 101.6763 57.404 0)
       (effects (font (size 1.27 1.27)) (justify left) hide)
     )
@@
     )
   )
-  (symbol (lib_id "fab:Screw_Terminal_01x03_P3.5mm") (at 91.2876 59.944 180) (unit 1)
-    (in_bom yes) (on_board yes) (dnp no) (fields_autoplaced)
-    (property "Reference" "J1" (at 91.2876 50.7492 0)
-      (effects (font (size 1.27 1.27)))
-    )
-    (property "Value" "Screw_Terminal_01x03_P3.5mm" (at 91.2876 53.2892 0)
-      (effects (font (size 1.27 1.27)))
-    )
-    (property "Footprint" "fab:TerminalBlock_OnShore_1x03_P3.50mm_Horizontal" (at 91.2876 59.944 0)
-      (effects (font (size 1.27 1.27)) hide)
-    )
-    (property "Datasheet" "www.on-shore.com/wp-content/uploads/ED555XDS.pdf" (at 91.2876 59.944 0)
+  (symbol (lib_id "fab:R") (at 166.243 101.219 270) (unit 1)
+    (in_bom yes) (on_board yes) (dnp no)
+    (property "Reference" "RRSW2" (at 163.703 96.901 90)
+      (effects (font (size 1.27 1.27)) (justify left))
+    )
+    (property "Value" "R499" (at 163.576 98.933 90)
+      (effects (font (size 1.27 1.27)) (justify left))
+    )
+    (property "Footprint" "fab:R_1206" (at 166.243 99.441 90)
+      (effects (font (size 1.27 1.27)) hide)
+    )
+    (property "Datasheet" "~" (at 166.243 101.219 0)
+      (effects (font (size 1.27 1.27)) hide)
+    )
+    (pin "1")
+    (pin "2")
+    (instances
+      (project "fla-lampi"
+        (path "/3934cdea-42c8-4ab1-b1be-2c4978ab08ae"
+          (reference "RRSW2") (unit 1)
+        )
+      )
+    )
+  )
+  (symbol (lib_id "fab:Conn_PinHeader_1x03_P2.54mm_Horizontal_SMD") (at 91.313 59.944 0) (unit 1)
+    (in_bom yes) (on_board yes) (dnp no)
+    (property "Reference" "J2" (at 91.313 51.816 0)
+      (effects (font (size 1.27 1.27)))
+    )
+    (property "Value" "Conn_PinHeader_1x03_P2.54mm_Horizontal_SMD" (at 82.169 48.26 0)
+      (effects (font (size 1.27 1.27)))
+    )
+    (property "Footprint" "fab:PinHeader_1x03_P2.54mm_Horizontal_SMD" (at 91.313 59.944 0)
+      (effects (font (size 1.27 1.27)) hide)
+    )
+    (property "Datasheet" "~" (at 91.313 59.944 0)
       (effects (font (size 1.27 1.27)) hide)
     )
@@
       (project "fla-lampi"
         (path "/3934cdea-42c8-4ab1-b1be-2c4978ab08ae"
-          (reference "J1") (unit 1)
-        )
-      )
-    )
-  )
-  (symbol (lib_id "fab:R") (at 166.243 101.219 270) (unit 1)
-    (in_bom yes) (on_board yes) (dnp no)
-    (property "Reference" "RRSW2" (at 163.703 96.901 90)
-      (effects (font (size 1.27 1.27)) (justify left))
-    )
-    (property "Value" "R499" (at 163.576 98.933 90)
-      (effects (font (size 1.27 1.27)) (justify left))
-    )
-    (property "Footprint" "fab:R_1206" (at 166.243 99.441 90)
-      (effects (font (size 1.27 1.27)) hide)
-    )
-    (property "Datasheet" "~" (at 166.243 101.219 0)
-      (effects (font (size 1.27 1.27)) hide)
-    )
-    (pin "1")
-    (pin "2")
-    (instances
-      (project "fla-lampi"
-        (path "/3934cdea-42c8-4ab1-b1be-2c4978ab08ae"
-          (reference "RRSW2") (unit 1)
+          (reference "J2") (unit 1)
         )
       )
@@
     )
   )
-  (symbol (lib_id "fab:Module_XIAO-RP2040_SocketSMD") (at 141.224 65.532 0) (unit 1)
+  (symbol (lib_id "fab:Module_XIAO-RP2040") (at 141.224 65.532 0) (unit 1)
     (in_bom yes) (on_board yes) (dnp no) (fields_autoplaced)
-    (property "Reference" "M1" (at 152.527 64.897 0)
-      (effects (font (size 1.27 1.27)) (justify left))
-    )
-    (property "Value" "Module_XIAO-RP2040_SocketSMD" (at 152.527 67.437 0)
-      (effects (font (size 1.27 1.27)) (justify left))
-    )
-    (property "Footprint" "fab:SeeedStudio_XIAO_SocketSMD" (at 141.224 65.532 0)
+    (property "Reference" "M2" (at 163.703 61.1439 0)
+      (effects (font (size 1.27 1.27)))
+    )
+    (property "Value" "Module_XIAO-RP2040" (at 163.703 63.6839 0)
+      (effects (font (size 1.27 1.27)))
+    )
+    (property "Footprint" "fab:SeeedStudio_XIAO_RP2040" (at 141.224 65.532 0)
       (effects (font (size 1.27 1.27)) hide)
     )
@@
     (pin "13")
     (pin "14")
+    (pin "15")
+    (pin "16")
+    (pin "17")
+    (pin "18")
+    (pin "19")
     (pin "2")
+    (pin "20")
     (pin "3")
     (pin "4")
@@
       (project "fla-lampi"
         (path "/3934cdea-42c8-4ab1-b1be-2c4978ab08ae"
-          (reference "M1") (unit 1)
-        )
-      )
-    )
-  )
-  (symbol (lib_id "fab:PWR_5V") (at 98.044 55.753 0) (unit 1)
+          (reference "M2") (unit 1)
+        )
+      )
+    )
+  )
+  (symbol (lib_id "fab:PWR_5V") (at 105.918 59.309 0) (unit 1)
     (in_bom yes) (on_board yes) (dnp no) (fields_autoplaced)
-    (property "Reference" "#PWR04" (at 98.044 59.563 0)
-      (effects (font (size 1.27 1.27)) hide)
-    )
-    (property "Value" "PWR_5V" (at 98.044 50.8 0)
-      (effects (font (size 1.27 1.27)))
-    )
-    (property "Footprint" "" (at 98.044 55.753 0)
-      (effects (font (size 1.27 1.27)) hide)
-    )
-    (property "Datasheet" "" (at 98.044 55.753 0)
+    (property "Reference" "#PWR04" (at 105.918 63.119 0)
+      (effects (font (size 1.27 1.27)) hide)
+    )
+    (property "Value" "PWR_5V" (at 105.918 54.864 0)
+      (effects (font (size 1.27 1.27)))
+    )
+    (property "Footprint" "" (at 105.918 59.309 0)
+      (effects (font (size 1.27 1.27)) hide)
+    )
+    (property "Datasheet" "" (at 105.918 59.309 0)
       (effects (font (size 1.27 1.27)) hide)
     )
@@
     )
   )
-  (symbol (lib_id "fab:Power_GND") (at 104.5464 61.976 0) (mirror y) (unit 1)
-    (in_bom yes) (on_board yes) (dnp no)
-    (property "Reference" "#PWR03" (at 104.5464 68.326 0)
-      (effects (font (size 1.27 1.27)) hide)
-    )
-    (property "Value" "Power_GND" (at 104.5464 66.294 0)
-      (effects (font (size 1.27 1.27)))
-    )
-    (property "Footprint" "" (at 104.5464 61.976 0)
-      (effects (font (size 1.27 1.27)) hide)
-    )
-    (property "Datasheet" "" (at 104.5464 61.976 0)
+  (symbol (lib_id "fab:Power_GND") (at 96.393 62.484 0) (unit 1)
+    (in_bom yes) (on_board yes) (dnp no)
+    (property "Reference" "#PWR03" (at 96.393 68.834 0)
+      (effects (font (size 1.27 1.27)) hide)
+    )
+    (property "Value" "GND" (at 99.822 63.627 0)
+      (effects (font (size 1.27 1.27)))
+    )
+    (property "Footprint" "" (at 96.393 62.484 0)
+      (effects (font (size 1.27 1.27)) hide)
+    )
+    (property "Datasheet" "" (at 96.393 62.484 0)
       (effects (font (size 1.27 1.27)) hide)
     )
@@
     )
   )
-  (symbol (lib_id "fab:Power_GND") (at 141.224 84.963 0) (mirror y) (unit 1)
-    (in_bom yes) (on_board yes) (dnp no)
-    (property "Reference" "#PWR09" (at 141.224 91.313 0)
-      (effects (font (size 1.27 1.27)) hide)
-    )
-    (property "Value" "Power_GND" (at 141.224 89.916 0)
-      (effects (font (size 1.27 1.27)))
-    )
-    (property "Footprint" "" (at 141.224 84.963 0)
-      (effects (font (size 1.27 1.27)) hide)
-    )
-    (property "Datasheet" "" (at 141.224 84.963 0)
-      (effects (font (size 1.27 1.27)) hide)
-    )
+  (symbol (lib_id "fab:Power_GND") (at 138.684 83.312 0) (mirror y) (unit 1)
+    (in_bom yes) (on_board yes) (dnp no)
+    (property "Reference" "#PWR09" (at 138.684 89.662 0)
+      (effects (font (size 1.27 1.27)) hide)
+    )
+    (property "Value" "Power_GND" (at 138.684 88.265 0)
+      (effects (font (size 1.27 1.27)))
+    )
+    (property "Footprint" "" (at 138.684 83.312 0)
+      (effects (font (size 1.27 1.27)) hide)
+    )
+    (property "Datasheet" "" (at 138.684 83.312 0)
+      (effects (font (size 1.27 1.27)) hide)
+    )

Commit message: Myndir
Other:
- moved on the sheet: J2, RRSW2, RSW1, SW1, SW2
